File: minionRVB.brd (EAGLE design)
At the start: 100.3 x 100 mm, 128 parts, among them IC1 74HCT245DW

Commit message: Update minionRVB
Parts:
- moved C59 69.2 mm to (58.1, 17.5), flipped to the bottom, turned to 90 degrees
- moved C60 63.2 mm to (53.7, 17.5), flipped to the bottom, turned to 90 degrees
- moved C57 60.2 mm to (49.2, 17.5), flipped to the bottom, turned to 90 degrees
- moved C55 60.0 mm to (58.1, 6.99), flipped to the bottom, turned to 90 degrees
- moved C54 54.7 mm to (53.7, 6.99), flipped to the bottom, turned to 90 degrees
- moved C58 54.4 mm to (44.8, 17.5), flipped to the bottom, turned to 90 degrees
- moved C53 49.5 mm to (49.2, 6.99), flipped to the bottom, turned to 90 degrees
- moved C56 49.0 mm to (44.8, 6.99), flipped to the bottom, turned to 90 degrees
- moved OUTPUT1 0.64 mm to (60.3, 8.89)
- moved OUTPUT8 0.64 mm to (60.3, 19.4)
- moved OUTPUT2 0.32 mm to (55.9, 8.89)
- moved OUTPUT7 0.32 mm to (55.9, 19.4)
Connections:
- net 5V: now also C53.2, C54.2, C55.2, C56.2, C57.2, C58.2, C59.2, C60.2
- net VCC: no longer C53.2, C54.2, C55.2, C56.2, C57.2, C58.2, C59.2, C60.2
Routing:
- net 5V: track 116.3 -> 124.7 mm
- net N$60: track 19.9 -> 19.3 mm
- net N$42: track 19.0 -> 18.4 mm
Other:
- outline, holes or cut-outs redrawn
